Commit message: Update the urdf robot

File: robotic_dog/urdf/robot.urdf (robot description, URDF)
Before this commit: robot full_robot, 13 links, 12 joints
Links:
- removed link part_1
- removed link part_1_10
- removed link part_1_11
- removed link part_1_12
- removed link part_1_13
- removed link part_1_2
- removed link part_1_3
- removed link part_1_4
- removed link part_1_5
- removed link part_1_6
- removed link part_1_7
- removed link part_1_8
- removed link part_1_9
- added link base_link, mass 5.79879; collision mesh filename=file:///home/pato/program_ws/src/robotic_dog/urdf/meshes/ba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; visual mesh filename=file:///home/pato/program_ws/src/robotic_dog/urdf/meshes/ba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
- added link hip_link1, mass 0.0639835; collision mesh filename=file:///home/pato/program_ws/src/robotic_dog/urdf/meshes/hi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; visual mesh filename=file:///home/pato/program_ws/src/robotic_dog/urdf/meshes/hi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
- added link hip_link2, mass 0.0639835; collision mesh filename=file:///home/pato/program_ws/src/robotic_dog/urdf/meshes/hi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; visual mesh filename=file:///home/pato/program_ws/src/robotic_dog/urdf/meshes/hi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
- added link hip_link3, mass 0.0639835; collision mesh filename=file:///home/pato/program_ws/src/robotic_dog/urdf/meshes/hi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; visual mesh filename=file:///home/pato/program_ws/src/robotic_dog/urdf/meshes/hi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
- added link hip_link4, mass 0.0639835; collision mesh filename=file:///home/pato/program_ws/src/robotic_dog/urdf/meshes/hi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; visual mesh filename=file:///home/pato/program_ws/src/robotic_dog/urdf/meshes/hi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
- added link shin_link1, mass 0.0626216; collision mesh filename=file:///home/pato/program_ws/src/robotic_dog/urdf/meshes/sh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; visual mesh filename=file:///home/pato/program_ws/src/robotic_dog/urdf/meshes/sh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
- added link shin_link1_2, mass 0.0626216; collision mesh filename=file:///home/pato/program_ws/src/robotic_dog/urdf/meshes/sh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; visual mesh filename=file:///home/pato/program_ws/src/robotic_dog/urdf/meshes/sh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
- added link shin_link2, mass 0.0626202; collision mesh filename=file:///home/pato/program_ws/src/robotic_dog/urdf/meshes/sh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; visual mesh filename=file:///home/pato/program_ws/src/robotic_dog/urdf/meshes/sh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
- added link shin_link2_2, mass 0.0626202; collision mesh filename=file:///home/pato/program_ws/src/robotic_dog/urdf/meshes/sh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; visual mesh filename=file:///home/pato/program_ws/src/robotic_dog/urdf/meshes/sh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
- added link thigh_link1, mass 0.0947343; collision mesh filename=file:///home/pato/program_ws/src/robotic_dog/urdf/meshes/th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; visual mesh filename=file:///home/pato/program_ws/src/robotic_dog/urdf/meshes/th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
- added link thigh_link1_2, mass 0.0947343; collision mesh filename=file:///home/pato/program_ws/src/robotic_dog/urdf/meshes/th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; visual mesh filename=file:///home/pato/program_ws/src/robotic_dog/urdf/meshes/th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
- added link thigh_link2, mass 0.0947331; collision mesh filename=file:///home/pato/program_ws/src/robotic_dog/urdf/meshes/th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; visual mesh filename=file:///home/pato/program_ws/src/robotic_dog/urdf/meshes/th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
- added link thigh_link2_2, mass 0.0947331; collision mesh filename=file:///home/pato/program_ws/src/robotic_dog/urdf/meshes/th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; visual mesh filename=file:///home/pato/program_ws/src/robotic_dog/urdf/meshes/th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
Joints:
- removed joint thig1
- removed joint thig2
- removed joint thig3
- removed joint thig4
- added joint thigh1: type revolute, parent hip_link1, child thigh_link1, origin xyz=0.0308937 0 -0.0095 rpy=-3.14159 1.5708 0, axis 0 0 1, limit lower=-3.141592653589793 upper=3.141592653589793 effort=10 velocity=10
- added joint thigh2: type revolute, parent hip_link3, child thigh_link1_2, origin xyz=0.0308937 -0 -0.0255 rpy=-0 -1.5708 0, axis 0 0 1, limit lower=-3.141592653589793 upper=3.141592653589793 effort=10 velocity=10
- added joint thigh3: type revolute, parent hip_link4, child thigh_link2, origin xyz=-0.0308937 -0 -0.0095 rpy=3.14159 -1.5708 0, axis 0 0 1, limit lower=-3.141592653589793 upper=3.141592653589793 effort=10 velocity=10
- added joint thigh4: type revolute, parent hip_link2, child thigh_link2_2, origin xyz=-0.0308937 0 -0.0255 rpy=-0 1.5708 0, axis 0 0 1, limit lower=-3.141592653589793 upper=3.141592653589793 effort=10 velocity=10
- joint hip1: child part_1_2 -> hip_link1; origin xyz=-0.0752765 0.115599 0.0877724 rpy=-0 1.5708 0 -> xyz=0.0733757 0.172834 0.214566 rpy=-1.5708 1.9718e-08 1.5708; parent part_1 -> base_link
- joint hip2: child part_1_5 -> hip_link3; origin xyz=-0.0752765 0.266599 0.0877724 rpy=-3.14159 -1.5708 0 -> xyz=-0.125624 0.172834 0.214566 rpy=1.5708 -0 1.5708; parent part_1 -> base_link
- joint hip3: child part_1_8 -> hip_link4; origin xyz=0.0787235 0.115599 0.0877724 rpy=-0 -1.5708 0 -> xyz=-0.125624 -0.0311657 0.214566 rpy=1.5708 -0 1.5708; parent part_1 -> base_link
- joint hip4: child part_1_11 -> hip_link2; origin xyz=0.0787235 0.266637 0.0877849 rpy=-3.14159 1.5708 0 -> xyz=0.0733757 -0.0311657 0.214566 rpy=-1.5708 -0 1.5708; parent part_1 -> base_link
- joint shin1: child part_1_4 -> shin_link1; origin xyz=0 -0.1 -0.015 rpy=0 -0 1.5708 -> xyz=0 -0.1 -0.0352 rpy=-0 -0 -0; parent part_1_3 -> thigh_link1
- joint shin2: child part_1_10 -> shin_link1_2; origin xyz=0 -0.1 -0.015 rpy=0 -0 1.5708 -> xyz=0 -0.1 -0.0352 rpy=0 -0 0; parent part_1_9 -> thigh_link1_2
- joint shin3: child part_1_13 -> shin_link2; origin xyz=0 -0.1 -0.015 rpy=0 -0 1.5708 -> xyz=0 0.1 -0.035 rpy=0 0 -0; parent part_1_12 -> thigh_link2
- joint shin4: child part_1_7 -> shin_link2_2; origin xyz=0 -0.1 -0.015 rpy=0 -0 1.5708 -> xyz=0 0.1 -0.035 rpy=0 0 -0; parent part_1_6 -> thigh_link2_2
